File: placa_robot/placa_robot.kicad_sch (KiCad schematic)
At the start: 1 part

Commit message: ultima prueba (creo que funciona)
Parts:
- added C1: C, symbol Device:C
Changed lines of the file:
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@@
+		)
+	)
+	(symbol
+		(lib_id "Device:C")
+		(at 152.4 78.74 0)
+		(unit 1)
+		(exclude_from_sim no)
+		(in_bom yes)
+		(on_board yes)
+		(dnp no)
+		(fields_autoplaced yes)
+		(property "Reference" "C1"
+			(at 156.21 77.4699 0)
+			(effects
+				(font
+					(size 1.27 1.27)
+				)
+				(justify left)
+			)
+		)
+		(property "Value" "C"
+			(at 156.21 80.0099 0)
+			(effects
+				(font
+					(size 1.27 1.27)
+				)
+				(justify left)
+			)
+		)
+		(property "Footprint" ""
+			(at 153.3652 82.55 0)
+			(effects
+				(font
+					(size 1.27 1.27)
+				)
+				(hide yes)
+			)
+		)
+		(property "Datasheet" "~"
+			(at 152.4 78.74 0)
+			(effects
+				(font
+					(size 1.27 1.27)
+				)
+				(hide yes)
+			)
+		)
+		(property "Description" "Unpolarized capacitor"
+			(at 152.4 78.74 0)
+			(effects
+				(font
+					(size 1.27 1.27)
+				)
+				(hide yes)
+			)
+		)
+		(pin "1"
+		)
+		(pin "2"
+		)
+		(instances
+			(project ""
+				(path "/8aa50d15-d96a-41b3-aa5f-664bff39212d"
+					(reference "C1")
+					(unit 1)
+				)
+			)
 		)
 	)

Commit message: librerias working
Parts:
- removed C1: C, symbol Device:C
- removed R1: R, symbol Device:R
- added IC1: MSP430FR2355TPT, MiSE:QFP50P900X900X160-48N, symbol MiSE:MSP430FR2355TPT
Changed lines of the file:
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@@
 	)
 	(symbol
-		(lib_id "Device:R")
-		(at 132.08 77.47 0)
+		(lib_id "MiSE:MSP430FR2355TPT")
+		(at 59.69 80.01 0)
 		(unit 1)
 		(exclude_from_sim no)
@@
 		(on_board yes)
 		(dnp no)
-		(fields_autoplaced yes)
-		(property "Reference" "R1"
-			(at 134.62 76.1999 0)
-			(effects
-				(font
-					(size 1.27 1.27)
-				)
-				(justify left)
-			)
-		)
-		(property "Value" "R"
-			(at 134.62 78.7399 0)
-			(effects
-				(font
-					(size 1.27 1.27)
-				)
-				(justify left)
-			)
-		)
-		(property "Footprint" ""
-			(at 130.302 77.47 90)
-			(effects
-				(font
-					(size 1.27 1.27)
-				)
-				(hide yes)
-			)
-		)
-		(property "Datasheet" "~"
-			(at 132.08 77.47 0)
-			(effects
-				(font
-					(size 1.27 1.27)
-				)
-				(hide yes)
-			)
-		)
-		(property "Description" "Resistor"
-			(at 132.08 77.47 0)
-			(effects
-				(font
-					(size 1.27 1.27)
-				)
-				(hide yes)
-			)
+		(property "Reference" "IC1"
+			(at 81.026 49.276 0)
+			(effects
+				(font
+					(size 1.27 1.27)
+				)
+			)
+		)
+		(property "Value" "MSP430FR2355TPT"
+			(at 81.026 51.816 0)
+			(effects
+				(font
+					(size 1.27 1.27)
+				)
+			)
+		)
+		(property "Footprint" "MiSE:QFP50P900X900X160-48N"
+			(at 185.42 134.29 0)
+			(effects
+				(font
+					(size 1.27 1.27)
+				)
+				(justify left top)
+				(hide yes)
+			)
+		)
+		(property "Datasheet" "https://datasheet.datasheetarchive.com/originals/distributors/DKDS41/DSANUWW0029426.pdf"
+			(at 185.42 234.29 0)
+			(effects
+				(font
+					(size 1.27 1.27)
+				)
+				(justify left top)
+				(hide yes)
+			)
+		)
+		(property "Description" "16-bit Microcontrollers - MCU 24MHz 105C ULP Microcontroller With 32 KB FRAM, 4 KB SRAM, 44 IO, 12-bit ADC, 12-bit DACs, OpAmp/PGA 48-LQFP -40 to 105"
+			(at 59.69 80.01 0)
+			(effects
+				(font
+					(size 1.27 1.27)
+				)
+				(hide yes)
+			)
+		)
+		(property "Height" "1.6"
+			(at 185.42 434.29 0)
+			(effects
+				(font
+					(size 1.27 1.27)
+				)
+				(justify left top)
+				(hide yes)
+			)
+		)
+		(property "Manufacturer_Name" "Texas Instruments"
+			(at 185.42 534.29 0)
+			(effects
+				(font
+					(size 1.27 1.27)
+				)
+				(justify left top)
+				(hide yes)
+			)
+		)
+		(property "Manufacturer_Part_Number" "MSP430FR2355TPT"
+			(at 185.42 634.29 0)
+			(effects
+				(font
+					(size 1.27 1.27)
+				)
+				(justify left top)
+				(hide yes)
+			)
+		)
+		(property "Mouser Part Number" "595-MSP430FR2355TPT"
+			(at 185.42 734.29 0)
+			(effects
+				(font
+					(size 1.27 1.27)
+				)
+				(justify left top)
+				(hide yes)
+			)
+		)
+		(property "Mouser Price/Stock" "https://www.mouser.co.uk/ProductDetail/Texas-Instruments/MSP430FR2355TPT?qs=gTYE2QTfZfTjQOKK%2F%2Fw59A%3D%3D"
+			(at 185.42 834.29 0)
+			(effects
+				(font
+					(size 1.27 1.27)
+				)
+				(justify left top)
+				(hide yes)
+			)
+		)
+		(property "Arrow Part Number" "MSP430FR2355TPT"
+			(at 185.42 934.29 0)
+			(effects
+				(font
+					(size 1.27 1.27)
+				)
+				(justify left top)
+				(hide yes)
+			)
+		)
+		(property "Arrow Price/Stock" "https://www.arrow.com/en/products/msp430fr2355tpt/texas-instruments?region=nac"
+			(at 185.42 1034.29 0)
+			(effects
+				(font
+					(size 1.27 1.27)
+				)
+				(justify left top)
+				(hide yes)
+			)
+		)
+		(pin "46"
+		)
+		(pin "16"
+		)
+		(pin "14"
+		)
+		(pin "8"
+		)
+		(pin "12"
+		)
+		(pin "40"
+		)
+		(pin "3"
+		)
+		(pin "41"
+		)
+		(pin "47"
+		)
+		(pin "18"
+		)
+		(pin "38"
+		)
+		(pin "4"
+		)
+		(pin "13"
+		)
+		(pin "6"
+		)
+		(pin "7"
 		)
 		(pin "1"
 		)
+		(pin "5"
+		)
+		(pin "9"
+		)
+		(pin "10"
+		)
+		(pin "48"
+		)
 		(pin "2"
+		)
+		(pin "11"
+		)
+		(pin "15"
+		)
+		(pin "17"
+		)
+		(pin "42"
+		)
+		(pin "45"
+		)
+		(pin "44"
+		)
+		(pin "19"
+		)
+		(pin "43"
+		)
+		(pin "20"
+		)
+		(pin "21"
+		)
+		(pin "39"
+		)
+		(pin "22"
+		)
+		(pin "24"
+		)
+		(pin "27"
+		)
+		(pin "30"
+		)
+		(pin "28"
+		)
+		(pin "26"
+		)
+		(pin "36"
+		)
+		(pin "23"
+		)
+		(pin "31"
+		)
+		(pin "35"
+		)
+		(pin "29"
+		)
+		(pin "33"
+		)
+		(pin "32"
+		)
+		(pin "25"
+		)
+		(pin "37"
+		)
+		(pin "34"
 		)
 		(instances
 			(project ""
 				(path "/8aa50d15-d96a-41b3-aa5f-664bff39212d"
-					(reference "R1")
+					(reference "IC1")
 					(unit 1)
 				)
-			)
-		)
-	)
-	(symbol
-		(lib_id "Device:C")
-		(at 152.4 78.74 0)
-		(unit 1)
-		(exclude_from_sim no)
-		(in_bom yes)
-		(on_board yes)
-		(dnp no)
-		(fields_autoplaced yes)
-		(property "Reference" "C1"
-			(at 156.21 77.4699 0)
-			(effects
-				(font
-					(size 1.27 1.27)
-				)
-				(justify left)
-			)
-		)
-		(property "Value" "C"
-			(at 156.21 80.0099 0)
-			(effects
-				(font
-					(size 1.27 1.27)
-				)
-				(justify left)
-			)
-		)
-		(property "Footprint" ""
-			(at 153.3652 82.55 0)
-			(effects
-				(font
-					(size 1.27 1.27)
-				)
-				(hide yes)
-			)
-		)
-		(property "Datasheet" "~"
-			(at 152.4 78.74 0)
-			(effects
-				(font
-					(size 1.27 1.27)
-				)
-				(hide yes)
-			)
-		)
-		(property "Description" "Unpolarized capacitor"
-			(at 152.4 78.74 0)
-			(effects
-				(font
-					(size 1.27 1.27)
-				)
-				(hide yes)
-			)
-		)
-		(pin "1"
-		)
-		(pin "2"
-		)
-		(instances
-			(project ""
-				(path "/8aa50d15-d96a-41b3-aa5f-664bff39212d"
-					(reference "C1")
-					(unit 1)
-				)
