File: placa_robot/untitled.kicad_sch (KiCad schematic)
At the start: 4 parts, among them Y1 Crystal

Commit message: Mas cosas
Parts:
- added C3: 100n, symbol Device:C
- added JP1: Jumper_2_Bridged, symbol Jumper:Jumper_2_Bridged
- C1, C2: value C -> 18p
Connections:
- net GND: now also LCD1.7 (K), C3.2
- net at LCD1.6 (A): now also JP1.1 (A)
- net VDD renamed +3.3V
- net +3.3V: now also C3.1, JP1.2 (B)
