File: placa_robot/untitled.kicad_sch (KiCad schematic)
At the start: 12 parts, among them U1 LMV324, U2 LMV324

Commit message: joystick
Parts:
- R1, R2, R3: value R -> 1K
Changed lines of the file:
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@@
 			)
 		)
-		(property "Value" "R"
+		(property "Value" "1K"
 			(at 86.36 44.4499 0)
 			(effects
@@
 		(on_board yes)
 		(dnp no)
-		(fields_autoplaced yes)
 		(property "Reference" "R1"
 			(at 86.36 86.3599 0)
@@
 			)
 		)
-		(property "Value" "R"
-			(at 86.36 88.8999 0)
+		(property "Value" "1K"
+			(at 86.36 89.154 0)
 			(effects
 				(font
@@
 			)
 		)
-		(property "Value" "R"
+		(property "Value" "1K"
 			(at 86.36 64.7699 0)
 			(effects
